File: demo7.sch (EAGLE design)
At the start: 11 parts, among them IC1 PIC18F46K22-I_P

Commit message: up
Parts:
- added COMMON: GND, pinhead:PINHD-1X1
- added SERIAL: UART1, pinhead:PINHD-1X2
Connections:
- new net N$1: IC1.RC6, SERIAL.2
- new net N$2: IC1.RC7, SERIAL.1
- net VSS: now also COMMON.1
Changed lines of the file:
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@@
 <?xml version="1.0" encoding="utf-8"?>
 <!DOCTYPE eagle SYSTEM "eagle.dtd">
-<eagle version="9.6.2">
+<eagle version="7.7.0">
 <drawing>
 <settings>
@@
 <parts>
 <part name="IC1" library="PIC18F46K22-I_P" deviceset="PIC18F46K22-I_P" device=""/>
-<part name="ICSP" library="con-lstb" library_urn="urn:adsk.eagle:library:162" deviceset="MA06-1" device="" package3d_urn="urn:adsk.eagle:package:8340/1" value="ICSP"/>
-<part name="VDD1" library="supply1" library_urn="urn:adsk.eagle:library:371" deviceset="VDD" device=""/>
-<part name="VDD2" library="supply1" library_urn="urn:adsk.eagle:library:371" deviceset="VDD" device=""/>
-<part name="VSS1" library="supply1" library_urn="urn:adsk.eagle:library:371" deviceset="VSS" device=""/>
-<part name="VSS2" library="supply1" library_urn="urn:adsk.eagle:library:371" deviceset="VSS" device=""/>
-<part name="R1" library="rcl" library_urn="urn:adsk.eagle:library:334" deviceset="R-US_" device="0204/7" package3d_urn="urn:adsk.eagle:package:23498/2" value="10K"/>
-<part name="VDD3" library="supply1" library_urn="urn:adsk.eagle:library:371" deviceset="VDD" device=""/>
-<part name="C1" library="rcl" library_urn="urn:adsk.eagle:library:334" deviceset="C-US" device="025-030X050" package3d_urn="urn:adsk.eagle:package:23631/1" value="0.1"/>
-<part name="C2" library="rcl" library_urn="urn:adsk.eagle:library:334" deviceset="C-US" device="025-030X050" package3d_urn="urn:adsk.eagle:package:23631/1" value="0.1"/>
-<part name="C3" library="rcl" library_urn="urn:adsk.eagle:library:334" deviceset="C-US" device="025-030X050" package3d_urn="urn:adsk.eagle:package:23631/1" value="10uf"/>
-<part name="C4" library="rcl" library_urn="urn:adsk.eagle:library:334" deviceset="C-US" device="025-030X050" package3d_urn="urn:adsk.eagle:package:23631/1" value="0.1"/>
-<part name="C5" library="rcl" library_urn="urn:adsk.eagle:library:334" deviceset="C-US" device="025-030X050" package3d_urn="urn:adsk.eagle:package:23631/1" value="10uf"/>
-<part name="VSS3" library="supply1" library_urn="urn:adsk.eagle:library:371" deviceset="VSS" device=""/>
-<part name="VSS4" library="supply1" library_urn="urn:adsk.eagle:library:371" deviceset="VSS" device=""/>
-<part name="VSS5" library="supply1" library_urn="urn:adsk.eagle:library:371" deviceset="VSS" device=""/>
-<part name="VSS6" library="supply1" library_urn="urn:adsk.eagle:library:371" deviceset="VSS" device=""/>
-<part name="VSS7" library="supply1" library_urn="urn:adsk.eagle:library:371" deviceset="VSS" device=""/>
-<part name="S1" library="switch-omron" library_urn="urn:adsk.eagle:library:377" deviceset="10-XX" device="" package3d_urn="urn:adsk.eagle:package:27496/1" value="RESET"/>
-<part name="VSS8" library="supply1" library_urn="urn:adsk.eagle:library:371" deviceset="VSS" device=""/>
-<part name="FRAME1" library="frames" library_urn="urn:adsk.eagle:library:229" deviceset="FRAME_A_L" device="" value="45(6)K22 demo board"/>
-<part name="R2" library="rcl" library_urn="urn:adsk.eagle:library:334" deviceset="R-US_" device="0204/7" package3d_urn="urn:adsk.eagle:package:23498/2" value="56 ohm"/>
-<part name="POWER" library="con-molex" library_urn="urn:adsk.eagle:library:165" deviceset="22-23-2021" device="" package3d_urn="urn:adsk.eagle:package:8078633/1" value="5VDC POWER"/>
-<part name="VSS9" library="supply1" library_urn="urn:adsk.eagle:library:371" deviceset="VSS" device=""/>
-<part name="VDD4" library="supply1" library_urn="urn:adsk.eagle:library:371" deviceset="VDD" device=""/>
+<part name="ICSP" library="con-lstb" deviceset="MA06-1" device="" value="ICSP"/>
+<part name="VDD1" library="supply1" deviceset="VDD" device=""/>
+<part name="VDD2" library="supply1" deviceset="VDD" device=""/>
+<part name="VSS1" library="supply1" deviceset="VSS" device=""/>
+<part name="VSS2" library="supply1" deviceset="VSS" device=""/>
+<part name="R1" library="rcl" deviceset="R-US_" device="0204/7" value="10K"/>
+<part name="VDD3" library="supply1" deviceset="VDD" device=""/>
+<part name="C1" library="rcl" deviceset="C-US" device="025-030X050" value="0.1"/>
+<part name="C2" library="rcl" deviceset="C-US" device="025-030X050" value="0.1"/>
+<part name="C3" library="rcl" deviceset="C-US" device="025-030X050" value="10uf"/>
+<part name="C4" library="rcl" deviceset="C-US" device="025-030X050" value="0.1"/>
+<part name="C5" library="rcl" deviceset="C-US" device="025-030X050" value="10uf"/>
+<part name="VSS3" library="supply1" deviceset="VSS" device=""/>
+<part name="VSS4" library="supply1" deviceset="VSS" device=""/>
+<part name="VSS5" library="supply1" deviceset="VSS" device=""/>
+<part name="VSS6" library="supply1" deviceset="VSS" device=""/>
+<part name="VSS7" library="supply1" deviceset="VSS" device=""/>
+<part name="S1" library="switch-omron" deviceset="10-XX" device="" value="RESET"/>
+<part name="VSS8" library="supply1" deviceset="VSS" device=""/>
+<part name="FRAME1" library="frames" deviceset="FRAME_A_L" device="" value="45(6)K22 demo board"/>
+<part name="R2" library="rcl" deviceset="R-US_" device="0204/7" value="56 ohm"/>
+<part name="POWER" library="con-molex" deviceset="22-23-2021" device="" value="5VDC POWER"/>
+<part name="VSS9" library="supply1" deviceset="VSS" device=""/>
+<part name="VDD4" library="supply1" deviceset="VDD" device=""/>
+<part name="COMMON" library="pinhead" deviceset="PINHD-1X1" device="" value="GND"/>
+<part name="SERIAL" library="pinhead" deviceset="PINHD-1X2" device="" value="UART1"/>
+<part name="VSS10" library="supply1" deviceset="VSS" device=""/>
 </parts>
 <sheets>
@@
 <instance part="VDD4" gate="G$1" x="69.85" y="80.01" smashed="yes" rot="R180">
 <attribute name="VALUE" x="71.12" y="77.47" size="1.778" layer="96"/>
+</instance>
+<instance part="COMMON" gate="G$1" x="132.08" y="25.4" smashed="yes">
+<attribute name="NAME" x="125.73" y="28.575" size="1.778" layer="95"/>
+<attribute name="VALUE" x="125.73" y="20.32" size="1.778" layer="96"/>
+</instance>
+<instance part="SERIAL" gate="G$1" x="132.08" y="12.7" smashed="yes">
+<attribute name="NAME" x="125.73" y="18.415" size="1.778" layer="95"/>
+<attribute name="VALUE" x="125.73" y="7.62" size="1.778" layer="96"/>
+</instance>
+<instance part="VSS10" gate="G$1" x="120.65" y="25.4" smashed="yes" rot="R270">
+<attribute name="VALUE" x="115.57" y="27.94" size="1.778" layer="96"/>
 </instance>
 </instances>
@@
 <junction x="69.85" y="85.09"/>
 </segment>
+<segment>
+<pinref part="COMMON" gate="G$1" pin="1"/>
+<wire x1="129.54" y1="25.4" x2="123.19" y2="25.4" width="0.1524" layer="91"/>
+<pinref part="VSS10" gate="G$1" pin="VSS"/>
+<wire x1="123.19" y1="25.4" x2="121.92" y2="25.4" width="0.1524" layer="91"/>
+<junction x="123.19" y="25.4"/>
+</segment>
 </net>
 <net name="MCLR_PIN" class="0">
@@
 </segment>
 </net>
+<net name="N$2" class="0">
+<segment>
+<pinref part="SERIAL" gate="G$1" pin="1"/>
+<wire x1="129.54" y1="15.24" x2="114.3" y2="15.24" width="0.1524" layer="91"/>
+<wire x1="114.3" y1="15.24" x2="114.3" y2="34.29" width="0.1524" layer="91"/>
+<pinref part="IC1" gate="G$1" pin="RC7"/>
+<wire x1="95.25" y1="34.29" x2="114.3" y2="34.29" width="0.1524" layer="91"/>
+<label x="101.6" y="35.56" size="1.778" layer="95"/>
+<label x="119.38" y="15.24" size="1.778" layer="95"/>
+</segment>
+</net>
+<net name="N$1" class="0">
+<segment>
+<pinref part="IC1" gate="G$1" pin="RC6"/>
+<wire x1="95.25" y1="31.75" x2="111.76" y2="31.75" width="0.1524" layer="91"/>
+<wire x1="111.76" y1="31.75" x2="111.76" y2="12.7" width="0.1524" layer="91"/>
+<pinref part="SERIAL" gate="G$1" pin="2"/>
+<wire x1="111.76" y1="12.7" x2="129.54" y2="12.7" width="0.1524" layer="91"/>
+<label x="101.6" y="33.02" size="1.778" layer="95"/>
+<label x="119.38" y="12.7" size="1.778" layer="95"/>
+</segment>
+</net>
 </nets>
 </sheet>
@@
 </schematic>
 </drawing>
-<compatibility>
-<note version="8.2" severity="warning">
-Since Version 8.2, EAGLE supports online libraries. The ids
-of those online libraries will not be understood (or retained)
-with this version.
-</note>
-<note version="8.3" severity="warning">
-Since Version 8.3, EAGLE supports URNs for individual library
-assets (packages, symbols, and devices). The URNs of those assets
-will not be understood (or retained) with this version.
-</note>
-<note version="8.3" severity="warning">
-Since Version 8.3, EAGLE supports the association of 3D packages
-with devices in libraries, schematics, and board files. Those 3D
-packages will not be understood (or retained) with this version.
-</note>
-<note version="8.4" severity="warning">
-Since Version 8.4, EAGLE supports properties for SPICE simulation.
-Probes in schematics and SPICE mapping objects found in parts and library devices
-will not be understood with this version. Update EAGLE to the latest version
-for full support of SPICE simulation.
-</note>
-</compatibility>
 </eagle>
