File: demo_46k22.brd (EAGLE design)
At the start: 86.3 x 100 mm, 11 parts, among them IC1 PIC18F46K22-I_P

Commit message: up
Parts:
- added COMMON: GND, pinhead:1X01
- added LED1: TLLG4400, led:LED3MM
- added R3: 900 ohm, rcl:0204/7
- added SERIAL: UART1, pinhead:1X02
Connections:
- new net N$1: IC1.25, SERIAL.2
- new net N$2: IC1.26, SERIAL.1
- new net N$3: IC1.38, R3.2
- net VSS: now also COMMON.1
Changed lines of the file:
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@@
 <attribute name="VALUE" x="86.36" y="76.2" size="1.016" layer="27" ratio="10"/>
+</element>
+<element name="COMMON" library="pinhead" library_urn="urn:adsk.eagle:library:325" package="1X01" package3d_urn="urn:adsk.eagle:package:22485/2" value="GND" x="22.86" y="-3.81" smashed="yes">
+<attribute name="NAME" x="21.5138" y="-1.9812" size="1.27" layer="25" ratio="10"/>
+<attribute name="POPULARITY" value="64" x="22.86" y="-3.81" size="1.778" layer="27" display="off"/>
+<attribute name="VALUE" x="21.59" y="-6.985" size="1.27" layer="27"/>
+</element>
+<element name="SERIAL" library="pinhead" library_urn="urn:adsk.eagle:library:325" package="1X02" package3d_urn="urn:adsk.eagle:package:22435/2" value="UART1" x="24.13" y="-8.89" smashed="yes">
+<attribute name="NAME" x="21.5138" y="-7.0612" size="1.27" layer="25" ratio="10"/>
+<attribute name="POPULARITY" value="98" x="24.13" y="-8.89" size="1.778" layer="27" display="off"/>
+<attribute name="VALUE" x="21.59" y="-12.065" size="1.27" layer="27"/>
+</element>
+<element name="R3" library="rcl" library_urn="urn:adsk.eagle:library:334" package="0204/7" package3d_urn="urn:adsk.eagle:package:23498/2" value="900 ohm" x="25.4" y="-16.51" smashed="yes">
+<attribute name="NAME" x="22.86" y="-15.2146" size="0.9906" layer="25" ratio="10"/>
+<attribute name="POPULARITY" value="48" x="25.4" y="-16.51" size="1.778" layer="27" display="off"/>
+<attribute name="SPICEPREFIX" value="R" x="25.4" y="-16.51" size="1.778" layer="27" display="off"/>
+<attribute name="VALUE" x="23.7744" y="-16.9926" size="0.9906" layer="27" ratio="10"/>
+</element>
+<element name="LED1" library="led" library_urn="urn:adsk.eagle:library:259" package="LED3MM" package3d_urn="urn:adsk.eagle:package:15797/1" value="TLLG4400" x="22.86" y="-20.32" smashed="yes">
+<attribute name="MF" value="VISHAY SEMICONDUCTOR" x="22.86" y="-20.32" size="1.778" layer="27" display="off"/>
+<attribute name="NAME" x="24.765" y="-19.939" size="1.27" layer="25" ratio="10"/>
+<attribute name="OC_FARNELL" value="1612435" x="22.86" y="-20.32" size="1.778" layer="27" display="off"/>
+<attribute name="POPULARITY" value="7" x="22.86" y="-20.32" size="1.778" layer="27" display="off"/>
+<attribute name="VALUE" x="24.765" y="-21.971" size="1.27" layer="27" ratio="10"/>
 </element>
 </elements>
@@
 <contactref element="S1" pad="4"/>
 <contactref element="POWER" pad="1"/>
+<contactref element="COMMON" pad="1"/>
+<wire x1="67.31" y1="93.98" x2="87.63" y2="81.28" width="0" layer="19" extent="1-1"/>
+<wire x1="46.99" y1="73.66" x2="67.31" y2="93.98" width="0" layer="19" extent="1-1"/>
+<wire x1="35.8394" y1="74.2188" x2="46.99" y2="73.66" width="0" layer="19" extent="1-1"/>
+<wire x1="35.8394" y1="80.7212" x2="35.8394" y2="74.2188" width="0" layer="19" extent="1-1"/>
+<wire x1="45.72" y1="43.18" x2="46.99" y2="73.66" width="0" layer="19" extent="1-1"/>
+<wire x1="38.1" y1="43.18" x2="45.72" y2="43.18" width="0" layer="19" extent="1-1"/>
+<wire x1="58.325" y1="40.64" x2="45.72" y2="43.18" width="0" layer="19" extent="1-1"/>
+<wire x1="73.755" y1="45.72" x2="58.325" y2="40.64" width="0" layer="19" extent="1-1"/>
+<wire x1="85.09" y1="48.26" x2="73.755" y2="45.72" width="0" layer="19" extent="1-1"/>
+<wire x1="91.44" y1="48.26" x2="85.09" y2="48.26" width="0" layer="19" extent="1-1"/>
+<wire x1="22.86" y1="-3.81" x2="38.1" y2="43.18" width="0" layer="19" extent="1-1"/>
 </signal>
 <signal name="MCLR_PIN">
@@
 <wire x1="58.3692" y1="68.58" x2="58.325" y2="68.58" width="0.1524" layer="1"/>
 </signal>
+<signal name="N$2">
+<contactref element="SERIAL" pad="1"/>
+<contactref element="IC1" pad="26"/>
+<wire x1="22.86" y1="-8.89" x2="73.755" y2="33.02" width="0" layer="19" extent="1-1"/>
+</signal>
+<signal name="N$1">
+<contactref element="IC1" pad="25"/>
+<contactref element="SERIAL" pad="2"/>
+<wire x1="25.4" y1="-8.89" x2="73.755" y2="30.48" width="0" layer="19" extent="1-1"/>
+</signal>
+<signal name="N$3">
+<contactref element="IC1" pad="38"/>
+<contactref element="R3" pad="2"/>
+<wire x1="29.21" y1="-16.51" x2="73.755" y2="63.5" width="0" layer="19" extent="1-1"/>
+</signal>
 </signals>
