File: demo_46k22.sch (EAGLE design)
At the start: 11 parts, among them IC1 PIC18F46K22-I_P

Commit message: up
Parts:
- added COMMON: GND, pinhead:PINHD-1X1
- added LED1: TLLG4400, led:TLLG4400
- added R3: 900 ohm, rcl:R-US_0204/7
- added SERIAL: UART1, pinhead:PINHD-1X2
Connections:
- new net N$1: IC1.RC6, SERIAL.2
- new net N$2: IC1.RC7, SERIAL.1
- new net N$3: IC1.RB5, R3.2
- net VSS: now also COMMON.1
Changed lines of the file:
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@@
 <part name="VSS9" library="supply1" library_urn="urn:adsk.eagle:library:371" deviceset="VSS" device=""/>
 <part name="VDD4" library="supply1" library_urn="urn:adsk.eagle:library:371" deviceset="VDD" device=""/>
+<part name="COMMON" library="pinhead" library_urn="urn:adsk.eagle:library:325" deviceset="PINHD-1X1" device="" package3d_urn="urn:adsk.eagle:package:22485/2" value="GND"/>
+<part name="SERIAL" library="pinhead" library_urn="urn:adsk.eagle:library:325" deviceset="PINHD-1X2" device="" package3d_urn="urn:adsk.eagle:package:22435/2" value="UART1"/>
+<part name="VSS10" library="supply1" library_urn="urn:adsk.eagle:library:371" deviceset="VSS" device=""/>
+<part name="R3" library="rcl" library_urn="urn:adsk.eagle:library:334" deviceset="R-US_" device="0204/7" package3d_urn="urn:adsk.eagle:package:23498/2" value="900 ohm"/>
+<part name="LED1" library="led" library_urn="urn:adsk.eagle:library:259" deviceset="TLLG4400" device="" package3d_urn="urn:adsk.eagle:package:15797/1"/>
 </parts>
 <sheets>
@@
 <instance part="VDD4" gate="G$1" x="69.85" y="80.01" smashed="yes" rot="R180">
 <attribute name="VALUE" x="71.12" y="77.47" size="1.778" layer="96"/>
+</instance>
+<instance part="COMMON" gate="G$1" x="132.08" y="25.4" smashed="yes">
+<attribute name="NAME" x="125.73" y="28.575" size="1.778" layer="95"/>
+<attribute name="VALUE" x="125.73" y="20.32" size="1.778" layer="96"/>
+</instance>
+<instance part="SERIAL" gate="G$1" x="132.08" y="12.7" smashed="yes">
+<attribute name="NAME" x="125.73" y="18.415" size="1.778" layer="95"/>
+<attribute name="VALUE" x="125.73" y="7.62" size="1.778" layer="96"/>
+</instance>
+<instance part="VSS10" gate="G$1" x="120.65" y="25.4" smashed="yes" rot="R270">
+<attribute name="VALUE" x="115.57" y="27.94" size="1.778" layer="96"/>
+</instance>
+<instance part="R3" gate="G$1" x="120.65" y="64.77" smashed="yes" rot="R180">
+<attribute name="NAME" x="119.38" y="63.2714" size="1.778" layer="95" rot="R180"/>
+<attribute name="VALUE" x="124.46" y="68.072" size="1.778" layer="96" rot="R180"/>
+</instance>
+<instance part="LED1" gate="G$1" x="129.54" y="66.04" smashed="yes" rot="R90">
+<attribute name="NAME" x="134.112" y="69.596" size="1.778" layer="95" rot="R180"/>
+<attribute name="VALUE" x="134.112" y="71.755" size="1.778" layer="96" rot="R180"/>
 </instance>
 </instances>
@@
 <junction x="69.85" y="85.09"/>
 </segment>
+<segment>
+<pinref part="COMMON" gate="G$1" pin="1"/>
+<wire x1="129.54" y1="25.4" x2="123.19" y2="25.4" width="0.1524" layer="91"/>
+<pinref part="VSS10" gate="G$1" pin="VSS"/>
+<wire x1="123.19" y1="25.4" x2="121.92" y2="25.4" width="0.1524" layer="91"/>
+<junction x="123.19" y="25.4"/>
+</segment>
 </net>
 <net name="MCLR_PIN" class="0">
@@
 </segment>
 </net>
+<net name="N$2" class="0">
+<segment>
+<pinref part="SERIAL" gate="G$1" pin="1"/>
+<wire x1="129.54" y1="15.24" x2="114.3" y2="15.24" width="0.1524" layer="91"/>
+<wire x1="114.3" y1="15.24" x2="114.3" y2="34.29" width="0.1524" layer="91"/>
+<pinref part="IC1" gate="G$1" pin="RC7"/>
+<wire x1="95.25" y1="34.29" x2="114.3" y2="34.29" width="0.1524" layer="91"/>
+<label x="101.6" y="35.56" size="1.778" layer="95"/>
+<label x="119.38" y="15.24" size="1.778" layer="95"/>
+</segment>
+</net>
+<net name="N$1" class="0">
+<segment>
+<pinref part="IC1" gate="G$1" pin="RC6"/>
+<wire x1="95.25" y1="31.75" x2="111.76" y2="31.75" width="0.1524" layer="91"/>
+<wire x1="111.76" y1="31.75" x2="111.76" y2="12.7" width="0.1524" layer="91"/>
+<pinref part="SERIAL" gate="G$1" pin="2"/>
+<wire x1="111.76" y1="12.7" x2="129.54" y2="12.7" width="0.1524" layer="91"/>
+<label x="101.6" y="33.02" size="1.778" layer="95"/>
+<label x="119.38" y="12.7" size="1.778" layer="95"/>
+</segment>
+</net>
+<net name="N$3" class="0">
+<segment>
+<pinref part="IC1" gate="G$1" pin="RB5"/>
+<pinref part="R3" gate="G$1" pin="2"/>
+<wire x1="115.57" y1="64.77" x2="95.25" y2="64.77" width="0.1524" layer="91"/>
+</segment>
+</net>
